Commit message: 更正lidar模型

File: autoware_gazebo/urdf/autoware_car.urdf (robot description, URDF)
Before this commit: robot autoware_car, 5 links, 4 joints
Joints:
- joint velodyne_link_joint: origin xyz=-0.47 0 1.55 rpy=0 0 1.58 -> xyz=-0.47 0 1.55 rpy=0 0 0

Commit message: lio-sam 3d slam 适配

File: autoware_gazebo/urdf/autoware_car.urdf (robot description, URDF)
Before this commit: robot autoware_car, 5 links, 4 joints
Joints:
- joint imu_link_joint: origin xyz=0 0 0.15 rpy=0 0 0 -> xyz=-0.47 0 1.55 rpy=0 0 0

Commit message: 1、cartographer源码引入 ； 2、整理autoware_slam包

File: autoware_gazebo/urdf/autoware_car.urdf (robot description, URDF)
Before this commit: robot autoware_car, 5 links, 4 joints
Links:
- removed link depth_camera_link
- removed link imu_link
- removed link velodyne_link
- added link gnss_link; visual box size=0.06 0.04 0.02
- added link tamagawa/imu_link; visual box size=0.06 0.04 0.02
- added link traffic_light_left_camera/camera_link; visual box size=0.06 0.04 0.02
- added link velodyne_top_base_link; visual cylinder length=0.0727 radius=0.052
Joints:
- removed joint depth_camera_link_joint
- removed joint imu_link_joint
- removed joint velodyne_link_joint
- added joint gnss_link_joint: type fixed, parent base_link, child gnss_link, origin xyz=0 0 0 rpy=0 0 0
- added joint tamagawa/imu_link_joint: type fixed, parent base_link, child tamagawa/imu_link, origin xyz=-0.47 0 1.55 rpy=0 0 0
- added joint traffic_light_left_camera/camera_link_joint: type fixed, parent base_link, child traffic_light_left_camera/camera_link, origin xyz=2.3 0 0.6 rpy=0 0 0
- added joint velodyne_top_base_link_joint: type fixed, parent base_link, child velodyne_top_base_link, origin xyz=-0.47 0 1.55 rpy=0 0 0

Commit message: 提高laser_scan高度，costmap能使用避障

File: autoware_gazebo/urdf/autoware_car.urdf (robot description, URDF)
Before this commit: robot autoware_car, 6 links, 5 joints
Joints:
- joint laser_link_joint: origin xyz=2.3 0 0.6 rpy=0 0 0 -> xyz=2.3 0 1.9 rpy=0 0 0
